Commit message: fixed mimic import issue

File: source/standalone/chiral/inspire_hand_isaac/handleft01151/urdf/handleft01151_test.urdf (robot description, URDF)
Before this commit: robot handleft01151, 19 links, 18 joints
Links:
- removed link Link11
- removed link Link12
- removed link Link13
- removed link Link14
- removed link Link15
- removed link Link16
- removed link Link17
- removed link Link18
- removed link Link19
- removed link Link20
- removed link Link21
- removed link Link22
- removed link link_LFTip1
- removed link link_LFTip2
- removed link link_LFTip3
- removed link link_LFTip4
- removed link link_LFTip5
- removed link world
- added link L_FF_L1, mass 0.1; collision mesh filename=package://handleft01151/meshes/Link15.STL; visual mesh filename=package://handleft01151/meshes/Link15.STL
- added link L_FF_L2, mass 0.1; collision mesh filename=package://handleft01151/meshes/Link16.STL; visual mesh filename=package://handleft01151/meshes/Link16.STL
- added link L_LF_L1, mass 0.1; collision mesh filename=package://handleft01151/meshes/Link21.STL; visual mesh filename=package://handleft01151/meshes/Link21.STL
- added link L_LF_L2, mass 0.1; collision mesh filename=package://handleft01151/meshes/Link22.STL; visual mesh filename=package://handleft01151/meshes/Link22.STL
- added link L_MF_L1, mass 0.1; collision mesh filename=package://handleft01151/meshes/Link17.STL; visual mesh filename=package://handleft01151/meshes/Link17.STL
- added link L_MF_L2, mass 0.1; collision mesh filename=package://handleft01151/meshes/Link18.STL; visual mesh filename=package://handleft01151/meshes/Link18.STL
- added link L_RF_L1, mass 0.1; collision mesh filename=package://handleft01151/meshes/Link19.STL; visual mesh filename=package://handleft01151/meshes/Link19.STL
- added link L_RF_L2, mass 0.1; collision mesh filename=package://handleft01151/meshes/Link20.STL; visual mesh filename=package://handleft01151/meshes/Link20.STL
- added link L_TH_L1, mass 0.1; collision mesh filename=package://handleft01151/meshes/Link11.STL; visual mesh filename=package://handleft01151/meshes/Link11.STL
- added link L_TH_L2, mass 0.1; collision mesh filename=package://handleft01151/meshes/Link12.STL; visual mesh filename=package://handleft01151/meshes/Link12.STL
- added link L_TH_L3, mass 0.1; collision mesh filename=package://handleft01151/meshes/Link13.STL; visual mesh filename=package://handleft01151/meshes/Link13.STL
- added link L_TH_L4, mass 0.1; collision mesh filename=package://handleft01151/meshes/Link14.STL; visual mesh filename=package://handleft01151/meshes/Link14.STL
- link base_link: mass 0.10331 -> 0.1
Joints:
- removed joint fixed
- removed joint joint011
- removed joint joint015
- removed joint joint017
- removed joint joint019
- removed joint joint021
- removed joint joint1112
- removed joint joint1213
- removed joint joint1314
- removed joint joint1516
- removed joint joint1718
- removed joint joint1920
- removed joint joint2122
- removed joint joint_LFTip1
- removed joint joint_LFTip2
- removed joint joint_LFTip3
- removed joint joint_LFTip4
- removed joint joint_LFTip5
- added joint L_FF_J1: type revolute, parent base_link, child L_FF_L1, origin xyz=0.0022853 -0.10493 0.032268 rpy=-0.034907 0 0, axis 0 0 -1, limit lower=0 upper=1.62 effort=50 velocity=1
- added joint L_FF_J2: type revolute, parent L_FF_L1, child L_FF_L2, origin xyz=-0.0024229 -0.032041 -0.001 rpy=0 0 0, axis 0 0 -1, limit lower=0 upper=1.82 effort=50, mimic joint=L_FF_J1 multiplier=1.13 offset=0
- added joint L_LF_J1: type revolute, parent base_link, child L_LF_L1, origin xyz=0.0022853 -0.10411 -0.025488 rpy=0.10472 0 0, axis 0 0 -1, limit lower=0 upper=1.62 effort=50 velocity=1
- added joint L_LF_J2: type revolute, parent L_LF_L1, child L_LF_L2, origin xyz=-0.0024229 -0.032041 -0.001 rpy=0 0 0, axis 0 0 -1, limit lower=0 upper=1.87 effort=50, mimic joint=L_LF_J1 multiplier=1.13 offset=0
- added joint L_MF_J1: type revolute, parent base_link, child L_MF_L1, origin xyz=0.0022853 -0.1055 0.01295 rpy=0 0 0, axis 0 0 -1, limit lower=0 upper=1.62 effort=50 velocity=1
- added joint L_MF_J2: type revolute, parent L_MF_L1, child L_MF_L2, origin xyz=-0.0024229 -0.032041 -0.001 rpy=0 0 0, axis 0 0 -1, limit lower=0 upper=1.75 effort=50, mimic joint=L_MF_J1 multiplier=1.13 offset=0
- added joint L_RF_J1: type revolute, parent base_link, child L_RF_L1, origin xyz=0.0022853 -0.10531 -0.0062872 rpy=0.05236 0 0, axis 0 0 -1, limit lower=0 upper=1.62 effort=50 velocity=1
- added joint L_RF_J2: type revolute, parent L_RF_L1, child L_RF_L2, origin xyz=-0.0024229 -0.032041 -0.001 rpy=0 0 0, axis 0 0 -1, limit lower=0 upper=1.75 effort=50, mimic joint=L_RF_J1 multiplier=1.08 offset=0
- added joint L_TH_J1: type revolute, parent base_link, child L_TH_L1, origin xyz=-0.01496 -0.0375 0.02045 rpy=1.5708 -1.5708 0, axis 0 0 1, limit lower=0 upper=1.30 effort=50 velocity=1
- added joint L_TH_J2: type revolute, parent L_TH_L1, child L_TH_L2, origin xyz=0.0099867 0.0098242 -0.0089 rpy=-1.5708 0 0.16939, axis 0 0 -1, limit lower=0 upper=0.68 effort=50 velocity=1
- added joint L_TH_J3: type revolute, parent L_TH_L2, child L_TH_L3, origin xyz=0.04407 -0.034553 -0.0008 rpy=0 0 0, axis 0 0 -1, limit lower=0 upper=0.77 effort=50, mimic joint=L_TH_J2 multiplier=1 offset=0
- added joint L_TH_J4: type revolute, parent L_TH_L3, child L_TH_L4, origin xyz=0.020248 -0.010156 -0.0012 rpy=0 0 0, axis 0 0 -1, limit lower=0 upper=0.597 effort=50, mimic joint=L_TH_J3 multiplier=1.13 offset=0

File: source/standalone/chiral/inspire_hand_isaac/handright01091/urdf/handright01091_test.urdf (robot description, URDF)
Before this commit: robot handright01091, 19 links, 18 joints
Links:
- removed link Link11
- removed link Link12
- removed link Link13
- removed link Link14
- removed link Link15
- removed link Link16
- removed link Link17
- removed link Link18
- removed link Link19
- removed link Link20
- removed link Link21
- removed link Link22
- removed link link_LFTip1
- removed link link_LFTip2
- removed link link_LFTip3
- removed link link_LFTip4
- removed link link_LFTip5
- removed link world
- added link R_FF_L1, mass 0.0042403; collision mesh filename=package://handright01091/meshes/Link15.STL; visual mesh filename=package://handright01091/meshes/Link15.STL
- added link R_FF_L2, mass 0.0045683; collision mesh filename=package://handright01091/meshes/Link16.STL; visual mesh filename=package://handright01091/meshes/Link16.STL
- added link R_LF_L1, mass 0.0042403; collision mesh filename=package://handright01091/meshes/Link21.STL; visual mesh filename=package://handright01091/meshes/Link21.STL
- added link R_LF_L2, mass 0.0035996; collision mesh filename=package://handright01091/meshes/Link22.STL; visual mesh filename=package://handright01091/meshes/Link22.STL
- added link R_MF_L1, mass 0.0042403; collision mesh filename=package://handright01091/meshes/Link17.STL; visual mesh filename=package://handright01091/meshes/Link17.STL
- added link R_MF_L2, mass 0.0050396; collision mesh filename=package://handright01091/meshes/Link18.STL; visual mesh filename=package://handright01091/meshes/Link18.STL
- added link R_RF_L1, mass 0.0042403; collision mesh filename=package://handright01091/meshes/Link19.STL; visual mesh filename=package://handright01091/meshes/Link19.STL
- added link R_RF_L2, mass 0.0045683; collision mesh filename=package://handright01091/meshes/Link20.STL; visual mesh filename=package://handright01091/meshes/Link20.STL
- added link R_TH_L1, mass 0.0018869; collision mesh filename=package://handright01091/meshes/Link11.STL; visual mesh filename=package://handright01091/meshes/Link11.STL
- added link R_TH_L2, mass 0.0066075; collision mesh filename=package://handright01091/meshes/Link12.STL; visual mesh filename=package://handright01091/meshes/Link12.STL
- added link R_TH_L3, mass 0.0037847; collision mesh filename=package://handright01091/meshes/Link13.STL; visual mesh filename=package://handright01091/meshes/Link13.STL
- added link R_TH_L4, mass 0.0033441; collision mesh filename=package://handright01091/meshes/Link14.STL; visual mesh filename=package://handright01091/meshes/Link14.STL
Joints:
- removed joint fixed
- removed joint joint011
- removed joint joint015
- removed joint joint017
- removed joint joint019
- removed joint joint021
- removed joint joint1112
- removed joint joint1213
- removed joint joint1314
- removed joint joint1516
- removed joint joint1718
- removed joint joint1920
- removed joint joint2122
- removed joint joint_LFTip1
- removed joint joint_LFTip2
- removed joint joint_LFTip3
- removed joint joint_LFTip4
- removed joint joint_LFTip5
- added joint R_FF_J1: type revolute, parent base_link, child R_FF_L1, origin xyz=0.0022853 -0.10493 -0.032268 rpy=-3.1067 0 0, axis 0 0 1, limit lower=0 upper=1.62 effort=50 velocity=1
- added joint R_FF_J2: type revolute, parent R_FF_L1, child R_FF_L2, origin xyz=-0.0026138 0.032026 -0.001 rpy=0 0 0, axis 0 0 1, limit lower=0 upper=1.82 effort=0, mimic joint=R_FF_J1 multiplier=1.13 offset=0
- added joint R_LF_J1: type revolute, parent base_link, child R_LF_L1, origin xyz=0.0022853 -0.10411 0.025488 rpy=3.0369 0 0, axis 0 0 1, limit lower=0 upper=1.62 effort=50 velocity=1
- added joint R_LF_J2: type revolute, parent R_LF_L1, child R_LF_L2, origin xyz=-0.0024229 0.032041 -0.001 rpy=0 0 0, axis 0 0 1, limit lower=0 upper=1.87 effort=50, mimic joint=R_LF_J1 multiplier=1.13 offset=0
- added joint R_MF_J1: type revolute, parent base_link, child R_MF_L1, origin xyz=0.0022853 -0.1055 -0.01295 rpy=-3.1416 0 0, axis 0 0 1, limit lower=0 upper=1.62 effort=50 velocity=1
- added joint R_MF_J2: type revolute, parent R_MF_L1, child R_MF_L2, origin xyz=-0.0024229 0.032041 -0.001 rpy=0 0 0, axis 0 0 1, limit lower=0 upper=1.75 effort=50, mimic joint=R_MF_J1 multiplier=1.13 offset=0
- added joint R_RF_J1: type revolute, parent base_link, child R_RF_L1, origin xyz=0.0022853 -0.10531 0.0062872 rpy=3.0892 0 0, axis 0 0 1, limit lower=0 upper=1.62 effort=50 velocity=1
- added joint R_RF_J2: type revolute, parent R_RF_L1, child R_RF_L2, origin xyz=-0.0024229 0.032041 -0.001 rpy=0 0 0, axis 0 0 1, limit lower=0 upper=1.75 effort=50, mimic joint=R_RF_J1 multiplier=1.08 offset=0
- added joint R_TH_J1: type revolute, parent base_link, child R_TH_L1, origin xyz=-0.01496 -0.0375 -0.02045 rpy=1.5708 -1.5708 0, axis 0 0 -1, limit lower=0 upper=1.30 effort=50 velocity=1
- added joint R_TH_J2: type revolute, parent R_TH_L1, child R_TH_L2, origin xyz=-0.0088099 0.010892 -0.00925 rpy=1.5708 0 2.8587, axis 0 0 1, limit lower=0 upper=0.68 effort=50 velocity=1
- added joint R_TH_J3: type revolute, parent R_TH_L2, child R_TH_L3, origin xyz=0.04407 0.034553 -0.0008 rpy=0 0 0, axis 0 0 1, limit lower=0 upper=0.77 effort=50, mimic joint=R_TH_J2 multiplier=1 offset=0
- added joint R_TH_J4: type revolute, parent R_TH_L3, child R_TH_L4, origin xyz=0.020248 0.010156 -0.0012 rpy=0 0 0, axis 0 0 1, limit lower=0 upper=0.597 effort=50, mimic joint=R_TH_J3 multiplier=1.13 offset=0

Commit message: move machine

File: source/standalone/chiral/inspire_hand_isaac/handleft01151/urdf/handleft01151_test.urdf (robot description, URDF)
Before this commit: robot handleft01151, 13 links, 12 joints
Links:
- added link root, mass 0.01
Joints:
- added joint fixed: type fixed, parent root, child base_link

File: source/standalone/chiral/inspire_hand_isaac/handright01091/urdf/handright01091_test.urdf (robot description, URDF)
Before this commit: robot handright01091, 13 links, 12 joints
Links:
- added link root
Joints:
- added joint fixed: type fixed, parent root, child base_link

Commit message: fixed more mimic joint issues

File: source/standalone/chiral/inspire_hand_isaac/handleft01151/urdf/handleft01151_test.urdf (robot description, URDF)
Before this commit: robot handleft01151, 14 links, 13 joints
Joints:
- joint L_FF_J2: limit lower=0 upper=1.82 effort=50 -> lower=-0.20 upper=2.0 effort=50
- joint L_LF_J2: limit lower=0 upper=1.87 effort=50 -> lower=-0.2 upper=2.1 effort=50
- joint L_MF_J2: limit lower=0 upper=1.75 effort=50 -> lower=-0.20 upper=1.90 effort=50
- joint L_RF_J2: limit lower=0 upper=1.75 effort=50 -> lower=-0.2 upper=1.9 effort=50
- joint L_TH_J3: limit lower=0 upper=0.77 effort=50 -> lower=-0.2 upper=0.8 effort=50
- joint L_TH_J4: limit lower=0 upper=0.597 effort=50 -> lower=-0.20 upper=0.85 effort=50

File: source/standalone/chiral/inspire_hand_isaac/handright01091/urdf/handright01091_test.urdf (robot description, URDF)
Before this commit: robot handright01091, 14 links, 13 joints
Joints:
- joint R_FF_J2: limit lower=0 upper=1.82 effort=0 -> lower=-0.2 upper=2.02 effort=0
- joint R_LF_J2: limit lower=0 upper=1.87 effort=50 -> lower=-0.2 upper=2.07 effort=50
- joint R_MF_J2: limit lower=0 upper=1.75 effort=50 -> lower=-0.2 upper=1.95 effort=50
- joint R_RF_J2: limit lower=0 upper=1.75 effort=50 -> lower=-0.2 upper=1.95 effort=50
- joint R_TH_J3: limit lower=0 upper=0.77 effort=50 -> lower=-0.2 upper=0.97 effort=50
- joint R_TH_J4: limit lower=0 upper=0.597 effort=50 -> lower=-0.2 upper=0.797 effort=50
